Commit message: Update starting positions and orientations. This will need to be changed in the wrapper as well (that generates the xacro file).

File: multi_ur_description/urdf/arm1g_transmission.urdf (robot description, URDF)
Before this commit: robot mutli_arm, 25 links, 24 joints
Joints:
- joint arm1base_joint: origin xyz=-2.0 -2.0 0.0 rpy=0 0 0.0 -> xyz=0 0 0.0 rpy=0 0 0.0
- joint arm2_base_joint: origin xyz=-2.2 -2.0 0.0 rpy=0 0 0.0 -> xyz=1.0 1.0 0.0 rpy=0 0 0.0

Commit message: Change starting position of one of the robot arms so they are closer together. This allows them to collide if moved in the correct orientation.

File: multi_ur_description/urdf/arm1g_transmission.urdf (robot description, URDF)
Before this commit: robot mutli_arm, 25 links, 24 joints
Joints:
- joint arm2_base_joint: origin xyz=1.0 1.0 0.0 rpy=0 0 0.0 -> xyz=0.2 0.2 0.0 rpy=0 0 0.0
