Commit message: Create script to start ROS pkg creation.
* Generate urdf based on a series of inputs from user when script is run
* Move xacro wrapper into script helper directory

File: src/test_double/urdf/test_double.urdf (robot description, URDF)
Before this commit: robot mutli_arm, 25 links, 24 joints
Links:
- removed link arm2_base
- removed link arm2_base_link
- removed link arm2_base_link_inertia
- removed link arm2_flange
- removed link arm2_forearm_link
- removed link arm2_ft_frame
- removed link arm2_shoulder_link
- removed link arm2_tool0
- removed link arm2_upper_arm_link
- removed link arm2_wrist_1_link
- removed link arm2_wrist_2_link
- removed link arm2_wrist_3_link
- added link robot2_base
- added link robot2_base_link
- added link robot2_base_link_inertia, mass 2.0; collision mesh filename=file:///home/roman/code/cps-gazebo-sim-2/install/multi_ur_d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; visual mesh filename=file:///home/roman/code/cps-gazebo-sim-2/install/multi_ur_d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
- added link robot2_flange
- added link robot2_forearm_link, mass 1.26; collision mesh filename=file:///home/roman/code/cps-gazebo-sim-2/install/multi_ur_d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; visual mesh filename=file:///home/roman/code/cps-gazebo-sim-2/install/multi_ur_d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
- added link robot2_ft_frame
- added link robot2_shoulder_link, mass 2.0; collision mesh filename=file:///home/roman/code/cps-gazebo-sim-2/install/multi_ur_d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; visual mesh filename=file:///home/roman/code/cps-gazebo-sim-2/install/multi_ur_d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
- added link robot2_tool0
- added link robot2_upper_arm_link, mass 3.42; collision mesh filename=file:///home/roman/code/cps-gazebo-sim-2/install/multi_ur_d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; visual mesh filename=file:///home/roman/code/cps-gazebo-sim-2/install/multi_ur_d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
- added link robot2_wrist_1_link, mass 0.8; collision mesh filename=file:///home/roman/code/cps-gazebo-sim-2/install/multi_ur_d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; visual mesh filename=file:///home/roman/code/cps-gazebo-sim-2/install/multi_ur_d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
- added link robot2_wrist_2_link, mass 0.8; collision mesh filename=file:///home/roman/code/cps-gazebo-sim-2/install/multi_ur_d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; visual mesh filename=file:///home/roman/code/cps-gazebo-sim-2/install/multi_ur_d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
- added link robot2_wrist_3_link, mass 0.35; collision mesh filename=file:///home/roman/code/cps-gazebo-sim-2/install/multi_ur_d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; visual mesh filename=file:///home/roman/code/cps-gazebo-sim-2/install/multi_ur_d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
Joints:
- removed joint arm2_base_joint
- removed joint arm2_base_link-base_fixed_joint
- removed joint arm2_base_link-base_link_inertia
- removed joint arm2_elbow_joint
- removed joint arm2_flange-tool0
- removed joint arm2_shoulder_lift_joint
- removed joint arm2_shoulder_pan_joint
- removed joint arm2_wrist_1_joint
- removed joint arm2_wrist_2_joint
- removed joint arm2_wrist_3-flange
- removed joint arm2_wrist_3_joint
- removed joint arm2_wrist_3_link-ft_frame
- added joint robot2_base_joint: type fixed, parent world, child robot2_base_link, origin xyz=0.2 0.2 0.0 rpy=0 0 0.0
- added joint robot2_base_link-base_fixed_joint: type fixed, parent robot2_base_link, child robot2_base, origin xyz=0 0 0 rpy=0 0 3.141592653589793
- added joint robot2_base_link-base_link_inertia: type fixed, parent robot2_base_link, child robot2_base_link_inertia, origin xyz=0 0 0 rpy=0 0 3.141592653589793
- added joint robot2_elbow_joint: type revolute, parent robot2_upper_arm_link, child robot2_forearm_link, origin xyz=-0.24355 0 0 rpy=0 0 0, axis 0 0 1, limit lower=-3.141592653589793 upper=3.141592653589793 effort=28.0 velocity=3.141592653589793
- added joint robot2_flange-tool0: type fixed, parent robot2_flange, child robot2_tool0, origin xyz=0 0 0 rpy=1.5707963267948966 0 1.5707963267948966
- added joint robot2_shoulder_lift_joint: type revolute, parent robot2_shoulder_link, child robot2_upper_arm_link, origin xyz=0 0 0 rpy=1.570796327 0 0, axis 0 0 1, limit lower=-6.283185307179586 upper=6.283185307179586 effort=56.0 velocity=3.141592653589793
- added joint robot2_shoulder_pan_joint: type revolute, parent robot2_base_link_inertia, child robot2_shoulder_link, origin xyz=0 0 0.15185 rpy=0 0 0, axis 0 0 1, limit lower=-6.283185307179586 upper=6.283185307179586 effort=56.0 velocity=3.141592653589793
- added joint robot2_wrist_1_joint: type revolute, parent robot2_forearm_link, child robot2_wrist_1_link, origin xyz=-0.2132 0 0.13105 rpy=0 0 0, axis 0 0 1, limit lower=-6.283185307179586 upper=6.283185307179586 effort=12.0 velocity=6.283185307179586
- added joint robot2_wrist_2_joint: type revolute, parent robot2_wrist_1_link, child robot2_wrist_2_link, origin xyz=0 -0.08535 -1.750557762378351e-11 rpy=1.570796327 0 0, axis 0 0 1, limit lower=-6.283185307179586 upper=6.283185307179586 effort=12.0 velocity=6.283185307179586
- added joint robot2_wrist_3-flange: type fixed, parent robot2_wrist_3_link, child robot2_flange, origin xyz=0 0 0 rpy=0 -1.5707963267948966 -1.5707963267948966
- added joint robot2_wrist_3_joint: type revolute, parent robot2_wrist_2_link, child robot2_wrist_3_link, origin xyz=0 0.0921 -1.8890025766262e-11 rpy=1.570796326589793 3.141592653589793 3.141592653589793, axis 0 0 1, limit lower=-6.283185307179586 upper=6.283185307179586 effort=12.0 velocity=6.283185307179586
- added joint robot2_wrist_3_link-ft_frame: type fixed, parent robot2_wrist_3_link, child robot2_ft_frame, origin xyz=0 0 0 rpy=3.141592653589793 0 0

File: src/test_double/urdf/test_double.urdf.xacro (robot description, xacro)
@@ -1,4 +1,4 @@
 <?xml version="1.0"?>
-<robot xmlns:xacro="http://wiki.ros.org/xacro" name="mutli_arm">
+<robot xmlns:xacro="http://wiki.ros.org/xacro" name="multi_arm">
   <!-- declare arguments -->
   <xacro:arg name="name"        default="arm1"/>
@@ -18,5 +18,5 @@
     </hardware>
     <!-- ARM 1 joints -->
-    <joint name="arm1shoulder_pan_joint">
+    <joint name="robot1_shoulder_pan_joint">
       <command_interface name="position"/>
       <command_interface name="velocity"/>
@@ -28,5 +28,5 @@
       <state_interface name="effort"/>
     </joint>
-    <joint name="arm1shoulder_lift_joint">
+    <joint name="robot1_shoulder_lift_joint">
       <command_interface name="position"/>
       <command_interface name="velocity"/>
@@ -38,5 +38,5 @@
       <state_interface name="effort"/>
     </joint>
-    <joint name="arm1elbow_joint">
+    <joint name="robot1_elbow_joint">
       <command_interface name="position"/>
       <command_interface name="velocity"/>
@@ -48,5 +48,5 @@
       <state_interface name="effort"/>
     </joint>
-    <joint name="arm1wrist_1_joint">
+    <joint name="robot1_wrist_1_joint">
       <command_interface name="position"/>
       <command_interface name="velocity"/>
@@ -58,5 +58,5 @@
       <state_interface name="effort"/>
     </joint>
-    <joint name="arm1wrist_2_joint">
+    <joint name="robot1_wrist_2_joint">
       <command_interface name="position"/>
       <command_interface name="velocity"/>
@@ -68,5 +68,5 @@
       <state_interface name="effort"/>
     </joint>
-    <joint name="arm1wrist_3_joint">
+    <joint name="robot1_wrist_3_joint">
       <command_interface name="position"/>
       <command_interface name="velocity"/>
@@ -79,5 +79,5 @@
     </joint>
     <!-- ARM 2 joints -->
-    <joint name="arm2_shoulder_pan_joint">
+    <joint name="robot2_shoulder_pan_joint">
       <command_interface name="position"/>
       <command_interface name="velocity"/>
@@ -89,5 +89,5 @@
       <state_interface name="effort"/>
     </joint>
-    <joint name="arm2_shoulder_lift_joint">
+    <joint name="robot2_shoulder_lift_joint">
       <command_interface name="position"/>
       <command_interface name="velocity"/>
@@ -99,5 +99,5 @@
       <state_interface name="effort"/>
     </joint>
-    <joint name="arm2_elbow_joint">
+    <joint name="robot2_elbow_joint">
       <command_interface name="position"/>
       <command_interface name="velocity"/>
@@ -109,5 +109,5 @@
       <state_interface name="effort"/>
     </joint>
-    <joint name="arm2_wrist_1_joint">
+    <joint name="robot2_wrist_1_joint">
       <command_interface name="position"/>
       <command_interface name="velocity"/>
@@ -119,5 +119,5 @@
       <state_interface name="effort"/>
     </joint>
-    <joint name="arm2_wrist_2_joint">
+    <joint name="robot2_wrist_2_joint">
       <command_interface name="position"/>
       <command_interface name="velocity"/>
@@ -129,5 +129,5 @@
       <state_interface name="effort"/>
     </joint>
-    <joint name="arm2_wrist_3_joint">
+    <joint name="robot2_wrist_3_joint">
       <command_interface name="position"/>
       <command_interface name="velocity"/>
@@ -157,5 +157,5 @@
   <xacro:ur_robot
     name="arm1"
-    tf_prefix="arm2_"
+    tf_prefix="robot2_"
     parent="world"
     joint_limits_parameters_file="$(find multi_ur_description)/config/$(arg ur_type)/joint_limits.yaml"
