Commit message: Small change to the wrapper file and original arm1g_transmison.urdf

File: scripts/helpers/robot_description_template.xacro (robot description, xacro)
@@ -1,4 +1,4 @@
 <?xml version="1.0"?>
-<robot xmlns:xacro="http://wiki.ros.org/xacro" name="mutli_arm">
+<robot xmlns:xacro="http://wiki.ros.org/xacro" name="multi_arm">
   <!-- declare arguments -->
   <xacro:arg name="name"        default="arm1"/>
@@ -79,5 +79,5 @@
     </joint>
     <!-- ARM 2 joints -->
-    <joint name="arm2_shoulder_pan_joint">
+  <joint name="arm2_shoulder_pan_joint">
       <command_interface name="position"/>
       <command_interface name="velocity"/>
@@ -89,5 +89,5 @@
       <state_interface name="effort"/>
     </joint>
-    <joint name="arm2_shoulder_lift_joint">
+  <joint name="arm2_shoulder_lift_joint">
       <command_interface name="position"/>
       <command_interface name="velocity"/>
@@ -99,5 +99,5 @@
       <state_interface name="effort"/>
     </joint>
-    <joint name="arm2_elbow_joint">
+  <joint name="arm2_elbow_joint">
       <command_interface name="position"/>
       <command_interface name="velocity"/>
@@ -109,5 +109,5 @@
       <state_interface name="effort"/>
     </joint>
-    <joint name="arm2_wrist_1_joint">
+  <joint name="arm2_wrist_1_joint">
       <command_interface name="position"/>
       <command_interface name="velocity"/>
@@ -119,5 +119,5 @@
       <state_interface name="effort"/>
     </joint>
-    <joint name="arm2_wrist_2_joint">
+  <joint name="arm2_wrist_2_joint">
       <command_interface name="position"/>
       <command_interface name="velocity"/>
@@ -129,5 +129,5 @@
       <state_interface name="effort"/>
     </joint>
-    <joint name="arm2_wrist_3_joint">
+  <joint name="arm2_wrist_3_joint">
       <command_interface name="position"/>
       <command_interface name="velocity"/>
@@ -156,5 +156,5 @@
   <!-- instantiate the second UR robot kinematic chain WITHOUT ros2_control -->
   <xacro:ur_robot
-    name="arm1"
+    name="arm2"
     tf_prefix="arm2_"
     parent="world"
